Commit message: add front camaera tf

File: src/go2_description/urdf/go2_description.urdf (robot description, URDF)
Before this commit: robot go2_description, 29 links, 28 joints
Links:
- added link Front_camera; visual cylinder length=0.01 radius=0.01
Joints:
- added joint Front_camera_joint: type fixed, parent Head_upper, child Front_camera, origin xyz=0.04 0 0.039 rpy=0 0 0, axis 0 0 0

Commit message: Add detected pose, optimize image threads

File: src/go2_description/urdf/go2_description.urdf (robot description, URDF)
Before this commit: robot go2_description, 30 links, 29 joints
Joints:
- joint Front_camera_joint: origin xyz=0.04 0 0.039 rpy=0 0 0 -> xyz=0.04 0 0.039 rpy=1.5708 0 1.5708

Commit message: Makes some clearly codes

File: src/go2_description/urdf/go2_description.urdf (robot description, URDF)
Before this commit: robot go2_description, 30 links, 29 joints
Joints:
- joint Front_camera_joint: origin xyz=0.04 0 0.039 rpy=1.5708 0 1.5708 -> xyz=0.04 0 0.039 rpy=0 0 0
